File: VCLFO_th_2.brd (EAGLE design)
At the start: 98.7 x 39.4 mm, 48 parts, among them IC1 LM358N, IC2 LM324N, IC3 LM358N, Q1 2N3904, Q2 2N3904

Commit message: Fixed circuit around timer vactrol (bypass diode for saw wave works better at high rates). Changed biggest timer cap + the bigger PSU caps from 1206 to TH electrolytics. Rerouted accordingly.
Parts:
- removed C4, C5: 10u, rcl:C1206
- added C10, C9: 10u, rcl:E2,5-5
- C1: value 10u -> 10u bipolar; device rcl:C1206 -> rcl:E2,5-5
- moved R1 16.5 mm to (69.8, 31.8), turned to 90 degrees
- moved PAD2 10.6 mm to (38.1, 29.2)
- moved R3 10.2 mm to (73.7, 31.8)
- moved D2 9.16 mm to (72.4, 53.3)
- moved D1 8.13 mm to (80.0, 53.3)
- moved PAD1 4.26 mm to (80.0, 46.4)
- moved C1 3.81 mm to (92.7, 31.8)
- moved C7 3.81 mm to (96.5, 31.8)
- moved R2 3.81 mm to (77.5, 31.8)
- moved C6 3.42 mm to (88.9, 36.2), turned to 180 degrees
- moved C2 1.80 mm to (63.5, 52.1), turned to 90 degrees
- moved C3 1.80 mm to (85.1, 52.1), turned to 270 degrees
Connections:
- removed net N$29: D3.C, R2.2
- new net N$2: D3.C, R17.2, R2.2
- net +12V: now also C9.+; no longer C4.1
- net -12V: now also C10.-; no longer C5.2
- net GND: now also C10.+, C9.-; no longer C4.2, C5.1
- net N$14: now also C1.+; no longer C1.1
- net SQR: no longer R17.2
- net TRI: now also C1.-; no longer C1.2
Routing:
- net N$2: track 0.00 -> 21.5 mm
- net N$29: track 14.0 -> 0.00 mm
- net N$24: track 17.1 -> 28.6 mm
- net N$5: track 13.6 -> 22.8 mm
- net -12V: track 95.0 -> 87.8 mm, vias 4 -> 2
- net N$1: track 73.0 -> 79.1 mm
- net +12V: track 81.3 -> 87.3 mm
- net N$13: track 16.3 -> 20.4 mm
- net N$19: track 13.6 -> 10.6 mm
- net TRI: track 130.1 -> 127.7 mm
- net N$14: track 4.95 -> 6.66 mm
- net N$11: track 7.62 -> 6.13 mm
- net SQR: track 104.5 -> 103.2 mm, vias 2 -> 1
Other:
- board text added: "C1 bipolar!"
- board text added: "v2.1 20160811 cc-by-sa 2016 Lars Bengtsson"
- board text removed: "v2 20160428 cc-by-sa 2016 Lars Bengtsson"

Commit message: Removed ledftover label on back of PCB. Changed footprint for vactrol LED to 5mm (easier to see polarity after manufacturing).
Parts:
- LED2: device led:LED3MM -> led:LED5MM
Changed lines of the file:
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@@
 <?xml version="1.0" encoding="utf-8"?>
 <!DOCTYPE eagle SYSTEM "eagle.dtd">
-<eagle version="7.5.0">
+<eagle version="7.7.0">
 <drawing>
 <settings>
@@
 <text x="31.75" y="59.055" size="1.016" layer="21" font="vector" ratio="10" rot="SR180">v2.1 20160811
 cc-by-sa 2016 Lars Bengtsson</text>
-<text x="3.81" y="26.67" size="1.016" layer="22" font="vector" ratio="1" rot="SMR90">VCLFO</text>
 <text x="21.59" y="22.86" size="1.016" layer="22" font="vector" ratio="10" rot="SMR90">cc-by-sa 2016 Lars Bengtsson</text>
 <wire x1="69.85" y1="59.69" x2="67.945" y2="59.69" width="0.254" layer="22"/>
@@
 <attribute name="VALUE" x="27.2034" y="56.5404" size="1.27" layer="27" ratio="10" rot="R90"/>
 </element>
-<element name="LED2" library="led" package="LED3MM" value="" x="63.5" y="25.4" smashed="yes" rot="R90">
+<element name="LED2" library="led" package="LED5MM" value="" x="63.5" y="25.4" smashed="yes" rot="R90">
 <attribute name="NAME" x="65.405" y="23.241" size="1.016" layer="25" ratio="10"/>
 <attribute name="VALUE" x="65.151" y="27.305" size="1.27" layer="27" ratio="10" rot="R90"/>
