File: VCLFO_th_2.sch (EAGLE design)
At the start: 48 parts, among them IC1 LM358N, IC2 LM324N, IC3 LM358N, Q1 2N3904, Q2 2N3904

Commit message: Fixed circuit around timer vactrol (bypass diode for saw wave works better at high rates). Changed biggest timer cap + the bigger PSU caps from 1206 to TH electrolytics. Rerouted accordingly.
Parts:
- removed C4, C5: 10u, rcl:C-USC1206
- added C10, C9: 10u, rcl:CPOL-USE2.5-5
- C1: value 10u -> 10u bipolar; device rcl:C-USC1206 -> rcl:CPOL-USE2.5-5
Connections:
- removed net N$29: D3.C, R2.2
- new net N$2: D3.C, R17.P$2, R2.2
- net +12V: now also C9.+; no longer C4.1
- net -12V: now also C10.-; no longer C5.2
- net GND: now also C10.+, C9.-; no longer C4.2, C5.1
- net N$14: now also C1.+; no longer C1.1
- net SQR: no longer R17.P$2
- net TRI: now also C1.-; no longer C1.2
Other:
- moved on the sheet: R2

Commit message: Removed ledftover label on back of PCB. Changed footprint for vactrol LED to 5mm (easier to see polarity after manufacturing).
Parts:
- LED2: device led:LED3MM -> led:LED5MM
Changed lines of the file:
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@@
 <?xml version="1.0" encoding="utf-8"?>
 <!DOCTYPE eagle SYSTEM "eagle.dtd">
-<eagle version="7.5.0">
+<eagle version="7.7.0">
 <drawing>
 <settings>
@@
 <part name="GND11" library="supply1" deviceset="GND" device=""/>
 <part name="GND13" library="supply1" deviceset="GND" device=""/>
-<part name="LED2" library="led" deviceset="LED" device="3MM"/>
+<part name="LED2" library="led" deviceset="LED" device="5MM"/>
 <part name="FRAME2" library="frames" deviceset="A3L-LOC" device=""/>
 <part name="S2" library="switch" deviceset="TL39PO" device="" value="SKS07SP"/>
